File: hardware/bike-odometer.kicad_pcb (KiCad board)
At the start: 2 copper layers, 26 parts, among them J1 Conn_ARM_JTAG_SWD_10, U1 nRF54L05-QFXX, U2 MLX92216, Y1 32 MHz, Y2 32.768 kHz

Commit message: Sourcing complete
Parts:
- added C14: 100n, Capacitor_SMD:C_0201_0603Metric, F.Cu at (159.9, 98.9)
- BT1: footprint Battery:BatteryHolder_Keystone_1060_1x2032 -> Battery:BatteryHolder_Renata_SMTU2032-LF_1x2032
- C1: footprint Capacitor_SMD:C_0402_1005Metric -> Capacitor_SMD:C_0603_1608Metric
- moved AE1 9.95 mm to (146.7, 80.7), turned to 45 degrees
Other:
- board outline added: 35 x 30 mm

Commit message: PCB placement
Parts:
- removed R1: 1k, Resistor_SMD:R_0201_0603Metric
- added H1: MountingHole, MountingHole:MountingHole_2.2mm_M2_ISO14580, F.Cu at (164.7, 85.8)
- added H2: MountingHole, MountingHole:MountingHole_2.2mm_M2_ISO14580, F.Cu at (139.7, 99.3)
- moved Y1 14.6 mm to (153.0, 85.9), turned to 180 degrees
- moved C13 13.8 mm to (156.2, 83.2), turned to 180 degrees
- moved U1 13.3 mm to (156.8, 91.6), turned to 90 degrees
- moved L1 11.3 mm to (151.5, 93.3), turned to 90 degrees
- moved U2 10.8 mm to (166.1, 91.2)
- moved C12 10.3 mm to (156.9, 85.1)
- moved AE1 10.1 mm to (156.6, 82.5), turned to 0 degrees
- moved L4 9.43 mm to (156.5, 84.2), turned to 90 degrees
- moved C14 9.17 mm to (164.9, 91.2)
- moved C5 8.52 mm to (160.8, 90.5), turned to -90 degrees
- moved FB1 7.59 mm to (150.8, 91.4), turned to 180 degrees
- moved C7 6.73 mm to (150.8, 90.6), turned to 180 degrees
- moved C1 6.70 mm to (151.5, 95.6), turned to 180 degrees
- moved C4 6.33 mm to (157.8, 95.6), turned to 180 degrees
- moved C11 6.31 mm to (156.0, 87.3), turned to -90 degrees
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Connections:
- C10 pad 1: Net-(U1-~{RESET}) -> Net-(J1-~{RESET})
- U1 pad 30: Net-(U1-~{RESET}) -> Net-(J1-~{RESET})
Routing:
- net GND: track 0.00 -> 6.12 mm
- net Net-(U1-XC1): track 0.00 -> 3.98 mm
- net Net-(U1-XC2): track 0.00 -> 3.80 mm
- net +BATT: track 0.00 -> 2.26 mm, vias 0 -> 1
- net Net-(U1-DECA): track 0.00 -> 1.21 mm
- net Net-(J1-~{RESET}): track 0.00 -> 1.14 mm
- added copper zone on B.Cu, net GND
- added copper zone on F.Cu, net GND
- added copper zone on In1.Cu, net GND
- added copper zone on In2.Cu, net GND
Other:
- board size 35 x 30 mm -> 32 x 26 mm
- copper layers 2 -> 4

Commit message: Layout
Parts:
- moved C13 0.69 mm to (156.9, 83.2), turned to 0 degrees
- moved C2 0.21 mm to (152.8, 94.1), turned to -90 degrees
- moved L1 0.21 mm to (151.5, 93.5), turned to -90 degrees
- moved C1 0.21 mm to (151.5, 95.4)
- moved C9 0.10 mm to (152.2, 91.5), turned to 180 degrees
- turned FB1 to 0 degrees
Connections:
- C1 pad 2: Net-(C1-Pad2) -> GND
- C2 pad 2: Net-(C1-Pad2) -> GND
- C3 pad 2: Net-(C1-Pad2) -> GND
- C4 pad 2: Net-(C1-Pad2) -> GND
- C5 pad 2: Net-(C1-Pad2) -> GND
- C6 pad 1: Net-(U1-DCC) -> Net-(U1-DECD)
- FB1 pad 1: Net-(U1-DCC) -> Net-(U1-DECD)
Routing:
- net Net-(U1-DECD): track 0.00 -> 5.67 mm, vias 0 -> 2
- net GND: track 6.12 -> 11.5 mm, vias 0 -> 7
- net Net-(U1-DECA): track 1.21 -> 5.57 mm, vias 0 -> 1
- net +BATT: track 2.26 -> 6.05 mm
- net Net-(U1-DCC): track 0.00 -> 3.08 mm
- net Net-(U1-P1.00): track 0.00 -> 1.64 mm
- net Net-(U1-P1.01): track 0.00 -> 1.48 mm
- net Net-(C12-Pad1): track 0.00 -> 1.19 mm
- net Net-(U1-ANT): track 0.00 -> 1.08 mm
- net Net-(C11-Pad1): track 0.00 -> 0.64 mm
Other:
- board size 32 x 26 mm -> 33 x 26 mm

Commit message: Layout complete
Parts:
- removed the U2 at (166.1, 91.2)
- added JP1: SolderJumper_2_Open, Jumper:SolderJumper-2_P1.3mm_Open_RoundedPad1.0x1.5mm, F.Cu at (163.9, 89.7)
- added JP2: SolderJumper_2_Bridged, Jumper:SolderJumper-2_P1.3mm_Bridged_RoundedPad1.0x1.5mm, F.Cu at (163.9, 92.3)
- added U1: DRV5034DG, Package_SON:Texas_X2SON-4-1EP_1.1x1.4mm_P0.5mm_EP0.8x0.6mm, F.Cu at (167.6, 90.0)
- moved C1 1.96 mm to (166.4, 90.0), turned to -90 degrees
- moved C8 0.07 mm to (156.9, 85.1)
- moved L2 0.05 mm to (156.6, 87.2)
- renumbered C14 to C1, C1 to C10, C2 to C11, C3 to C12, C4 to C13, C5 to C14, C10 to C2, C6 to C3, C9 to C4, C8 to C5, C11 to C6, C12 to C8, C13 to C9, U1 to U2
Connections:
- AE1 pad 2: (no net) -> GND
- C2 pad 1: Net-(J1-~{RESET}) -> Net-(U2-~{RESET})
- J1 pad 10: Net-(J1-~{RESET}) -> unconnected-(J1-~{RESET}-Pad10)
- U2 pad 30: Net-(J1-~{RESET}) -> Net-(U2-~{RESET})
Routing:
- net +BATT: track 6.05 -> 58.5 mm, vias 1 -> 6
- net Net-(J1-SWDIO/TMS): track 0.00 -> 19.5 mm, vias 0 -> 2
- net Net-(J1-SWCLK/TCK): track 0.00 -> 17.3 mm, vias 0 -> 2
- net GND: track 11.5 -> 28.1 mm, vias 7 -> 50
- net /hall_sensor: track 0.00 -> 6.94 mm
- net Net-(U2-DECA): track 5.57 -> 12.2 mm, vias 1 -> 2
- net Net-(JP2-A): track 0.00 -> 4.36 mm
- net Net-(JP1-A): track 0.00 -> 3.98 mm
- net Net-(AE1-A): track 0.00 -> 1.31 mm
- net Net-(U2-~{RESET}): track 0.00 -> 1.14 mm
- net Net-(J1-~{RESET}): track 1.14 -> 0.00 mm
- net Net-(C6-Pad1): track 0.64 -> 1.25 mm

Commit message: Generate gerbers with CI
Other:
- board text added: "<<hash>>"
Changed lines of the file:
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@@
 			(outputformat 1)
 			(mirror no)
-			(drillshape 1)
+			(drillshape 0)
 			(scaleselection 1)
-			(outputdirectory "")
+			(outputdirectory "gbr/")
 		)
 	)
@@
 		(layer "Edge.Cuts")
 	)
+	(gr_text "<<hash>>"
+		(at 151.9 84 0)
+		(layer "B.SilkS")
+		(effects
+			(font
+				(size 1 1)
+				(thickness 0.1)
+			)
+			(justify bottom mirror)
+		)
+	)
 	(segment
