File: hardware/bike-odometer.kicad_pcb (KiCad board)
At the start: 4 copper layers, 33 x 26 mm, 30 parts, among them J1 Conn_ARM_JTAG_SWD_10, U1 DRV5034DG, U2 nRF54L05-QFXX, Y1 32 MHz, Y2 32.768 kHz

Commit message: Revised PCB mounting hole positions
Parts:
- removed JP1: SolderJumper_2_Open, Jumper:SolderJumper-2_P1.3mm_Open_RoundedPad1.0x1.5mm
- removed JP2: SolderJumper_2_Bridged, Jumper:SolderJumper-2_P1.3mm_Bridged_RoundedPad1.0x1.5mm
- U1: value DRV5034DG -> DRV5032DG
- moved H1 1.00 mm to (165.7, 85.8)
- moved H2 1.00 mm to (138.7, 99.3)
Connections:
- U1 pad 3: Net-(JP2-A) -> /hall_sensor
- U1 pad 4: Net-(JP1-A) -> unconnected-(U1-OUT1-Pad4)
Routing:
- net Net-(JP2-A): track 4.36 -> 0.00 mm
- net Net-(JP1-A): track 3.98 -> 0.00 mm
- net /hall_sensor: track 6.94 -> 10.5 mm
